Commit message: Adjust base height in URDF to improve robot stability

File: fws_robot_description/robots/fws_robot.urdf.xacro (robot description, xacro)
@@ -20,5 +20,5 @@
   <link name="base_footprint"/> <!--link name="base_footprint"/ -->
   <xacro:base_v0 parent="base_footprint"> <!-- xacro:base_v0 parent="base_footprint" -->
-	<origin xyz="0 0 0"/>
+	<origin xyz="0 0 0.250"/>
   </xacro:base_v0>
   <!-- lidar_base -->

Commit message: Adjust lidar_base origin height for improved sensor positioning

File: fws_robot_description/robots/fws_robot.urdf.xacro (robot description, xacro)
@@ -24,5 +24,5 @@
   <!-- lidar_base -->
   <xacro:lidar_base_v0 parent="base_link">
-	<origin xyz="-0.022 0 0.035"/>
+	<origin xyz="-0.022 0 0.005"/>
   </xacro:lidar_base_v0>
   <!-- lidar_head -->

Commit message: Add inrof_field mesh and update URDF for fws_robot
- Added new STL file for inrof_field mesh to the project.
- Updated the base origin position in fws_robot.urdf.xacro to (0, 0, 0).
- Adjusted lidar_base origin position in fws_robot.urdf.xacro from (0.005) to (0.035).
- Initialized gz_ros2_control as a subproject.

File: fws_robot_description/robots/fws_robot.urdf.xacro (robot description, xacro)
@@ -20,9 +20,9 @@
   <link name="base_footprint"/> <!--link name="base_footprint"/ -->
   <xacro:base_v0 parent="base_footprint"> <!-- xacro:base_v0 parent="base_footprint" -->
-	<origin xyz="0 0 0.250"/>
+	<origin xyz="0 0 0"/>
   </xacro:base_v0>
   <!-- lidar_base -->
   <xacro:lidar_base_v0 parent="base_link">
-	<origin xyz="-0.022 0 0.005"/>
+	<origin xyz="-0.022 0 0.035"/>
   </xacro:lidar_base_v0>
   <!-- lidar_head -->
